Commit message: fix(I-016/BUG-1): extend LiDAR from 180° to 360°, add contact sensor
LiDAR was configured min_angle=-π/2 to max_angle=π/2 (only frontal 180°).
Robot was completely blind behind and beyond 90° to each side — any escape
reverse maneuver (backward motion) had zero LiDAR coverage.

- walle.urdf.xacro: LiDAR min_angle=-π, max_angle=π (full 360°)
- Increase samples 720→1080 to maintain ~0.33°/sample resolution
- Add contact/bumper sensor on base_link (topic: /bumper) as last-resort
  safety net when LiDAR fails to prevent a collision

Co-Authored-By: Claude Sonnet 4.6 <noreply@anthropic.com>

File: walle_ws/src/walle_description/urdf/walle.urdf.xacro (robot description, xacro)
@@ -473,8 +473,8 @@
         <scan>
           <horizontal>
-            <samples>720</samples>
+            <samples>1080</samples>
             <resolution>1</resolution>
-            <min_angle>-1.57079632679</min_angle>
-            <max_angle>1.57079632679</max_angle>
+            <min_angle>-3.14159265359</min_angle>
+            <max_angle>3.14159265359</max_angle>
           </horizontal>
         </scan>
@@ -495,3 +495,16 @@
     </sensor>
   </gazebo>
+  <!-- Contact/bumper sensor — last-resort safety net (BUG-4 fix) -->
+  <gazebo reference="base_link">
+    <sensor name="bumper" type="contact">
+      <always_on>true</always_on>
+      <update_rate>30.0</update_rate>
+      <contact>
+        <collision>base_link_collision</collision>
+      </contact>
+      <plugin filename="gz-sim-contact-system" name="gz::sim::systems::Contact">
+        <topic>/bumper</topic>
+      </plugin>
+    </sensor>
+  </gazebo>
 </robot>
